File: pcb/pcb.kicad_pcb (KiCad board)
At the start: 2 copper layers, 100 x 74 mm, 135 parts, among them CN2 HC-XH-2A-G, CN3 HC-XH-2A-G, CN4 HC-XH-2A-G, CN5 HC-XH-2A-G, CN6 HC-XH-2A-G, CN7 HC-XH-6A-G, CN8 HC-XH-4A-G, CN9 HC-XH-2A-G, J1 Conn_01x04_Male, J12 FAN_D858, J13 Load, J15 PWR_T12, J18 24v, J2 220, J20 POWER_BTN, J22 FAN_24V, J3 POWER_BTN_MCU, J4 220_OUT, J7 JP1, J8 JP2, J9 PWR_D907, Q1 IRFR5505TR, Q10 IRFR5505TR, Q11 2n3904S-RTK_PS_C18536, Q2 2n3904S-RTK_PS_C18536, Q3 IRFR5505TR, Q4 BTA16-600B, Q5 2n3904S-RTK_PS_C18536, Q6 IRFR5505TR, Q7 2n3904S-RTK_PS_C18536, Q8 2n3904S-RTK_PS_C18536, Q9 BCX56, U1 FM24C64B, U2 STM32F103CBTx, U3 TL431D, U4 AD8541AKSZ-REEL7, U5 AD8541AKSZ-REEL7, U6 MOC3041M, U7 AD8541AKSZ-REEL7, U8 MC34063AD, U9 H11AA1, Y1 Crystal_GND24

Commit message: Change resistense on R46 to 1k (add raleay on more power)
Parts:
- R46: value 10k -> 1k
Changed lines of the file:
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@@
         (effects (font (size 1 1) (thickness 0.15)))
     )
-    (fp_text value "10k" (at 0 1.82 90) (layer "F.Fab")
+    (fp_text value "1k" (at 0 1.82 90) (layer "F.Fab")
         (effects (font (size 1 1) (thickness 0.15)))
     )
@@
     (descr "Resistor SMD 1206 (3216 Metric), square (rectangular) end terminal, IPC_7351 nominal with elongated pad for handsoldering. (Body size source: IPC-SM-782 page 72, https://www.pcb-3d.com/wordpress/wp-content/uploads/ipc-sm-782a_amendment_1_and_2.pdf), generated with kicad-footprint-generator")
     (tags "resistor handsolder")
-    (property "Sheetfile" "qsolder_pcb.kicad_sch")
+    (property "Sheetfile" "pcb.kicad_sch")
     (property "Sheetname" "")
     (property "ki_description" "Resistor")
@@
     (descr "Capacitor SMD 1206 (3216 Metric), square (rectangular) end terminal, IPC_7351 nominal with elongated pad for handsoldering. (Body size source: IPC-SM-782 page 76, https://www.pcb-3d.com/wordpress/wp-content/uploads/ipc-sm-782a_amendment_1_and_2.pdf), generated with kicad-footprint-generator")
     (tags "capacitor handsolder")
-    (property "Sheetfile" "qsolder_pcb.kicad_sch")
+    (property "Sheetfile" "pcb.kicad_sch")
     (property "Sheetname" "")
     (property "ki_description" "Unpolarized capacitor")
@@
     (descr "Resistor SMD 1206 (3216 Metric), square (rectangular) end terminal, IPC_7351 nominal with elongated pad for handsoldering. (Body size source: IPC-SM-782 page 72, https://www.pcb-3d.com/wordpress/wp-content/uploads/ipc-sm-782a_amendment_1_and_2.pdf), generated with kicad-footprint-generator")
     (tags "resistor handsolder")
-    (property "Sheetfile" "qsolder_pcb.kicad_sch")
+    (property "Sheetfile" "pcb.kicad_sch")
     (property "Sheetname" "")
     (property "ki_description" "Resistor")
@@
     (descr "Capacitor SMD 1206 (3216 Metric), square (rectangular) end terminal, IPC_7351 nominal with elongated pad for handsoldering. (Body size source: IPC-SM-782 page 76, https://www.pcb-3d.com/wordpress/wp-content/uploads/ipc-sm-782a_amendment_1_and_2.pdf), generated with kicad-footprint-generator")
     (tags "capacitor handsolder")
-    (property "Sheetfile" "qsolder_pcb.kicad_sch")
+    (property "Sheetfile" "pcb.kicad_sch")
     (property "Sheetname" "")
     (property "ki_description" "Unpolarized capacitor")
@@
     (descr "Capacitor SMD 1206 (3216 Metric), square (rectangular) end terminal, IPC_7351 nominal with elongated pad for handsoldering. (Body size source: IPC-SM-782 page 76, https://www.pcb-3d.com/wordpress/wp-content/uploads/ipc-sm-782a_amendment_1_and_2.pdf), generated with kicad-footprint-generator")
     (tags "capacitor handsolder")
-    (property "Sheetfile" "qsolder_pcb.kicad_sch")
+    (property "Sheetfile" "pcb.kicad_sch")
     (property "Sheetname" "")
     (property "ki_description" "Unpolarized capacitor")
@@
     (descr "Through hole straight socket strip, 1x04, 2.54mm pitch, single row (from Kicad 4.0.7), script generated")
     (tags "Through hole socket strip THT 1x04 2.54mm single row")
-    (property "Sheetfile" "qsolder_pcb.kicad_sch")
+    (property "Sheetfile" "pcb.kicad_sch")
     (property "Sheetname" "")
     (property "ki_description" "Generic connector, single row, 01x04, script generated (kicad-library-utils/schlib/autogen/connector/)")
@@
     (descr "SOIC, 8 Pin (JEDEC MS-012AA, https://www.analog.com/media/en/package-pcb-resources/package/pkg_pdf/soic_narrow-r/r_8.pdf), generated with kicad-footprint-generator ipc_gullwing_generator.py")
     (tags "SOIC SO")
-    (property "Sheetfile" "qsolder_pcb.kicad_sch")
+    (property "Sheetfile" "pcb.kicad_sch")
     (property "Sheetname" "")
     (property "ki_description" "Shunt Regulator, SO-8")
@@
     (descr "Resistor SMD 1206 (3216 Metric), square (rectangular) end terminal, IPC_7351 nominal with elongated pad for handsoldering. (Body size source: IPC-SM-782 page 72, https://www.pcb-3d.com/wordpress/wp-content/uploads/ipc-sm-782a_amendment_1_and_2.pdf), generated with kicad-footprint-generator")
     (tags "resistor handsolder")
-    (property "Sheetfile" "qsolder_pcb.kicad_sch")
+    (property "Sheetfile" "pcb.kicad_sch")
     (property "Sheetname" "")
     (property "ki_description" "Resistor")
@@
     (descr "Capacitor SMD 1206 (3216 Metric), square (rectangular) end terminal, IPC_7351 nominal with elongated pad for handsoldering. (Body size source: IPC-SM-782 page 76, https://www.pcb-3d.com/wordpress/wp-content/uploads/ipc-sm-782a_amendment_1_and_2.pdf), generated with kicad-footprint-generator")
     (tags "capacitor handsolder")
-    (property "Sheetfile" "qsolder_pcb.kicad_sch")
+    (property "Sheetfile" "pcb.kicad_sch")
     (property "Sheetname" "")
     (property "ki_description" "Unpolarized capacitor")
@@
     (descr "SMD Crystal SERIES SMD2520/4 http://www.icbase.com/File/PDF/HKC/HKC00061008.pdf, 5.0x3.2mm^2 package")
     (tags "SMD SMT crystal")
-    (property "Sheetfile" "qsolder_pcb.kicad_sch")
+    (property "Sheetfile" "pcb.kicad_sch")
     (property "Sheetname" "")
     (property "ki_description" "Four pin crystal, GND on pins 2 and 4")
@@
     (descr "Resistor SMD 1206 (3216 Metric), square (rectangular) end terminal, IPC_7351 nominal with elongated pad for handsoldering. (Body size source: IPC-SM-782 page 72, https://www.pcb-3d.com/wordpress/wp-content/uploads/ipc-sm-782a_amendment_1_and_2.pdf), generated with kicad-footprint-generator")
     (tags "resistor handsolder")
-    (property "Sheetfile" "qsolder_pcb.kicad_sch")
+    (property "Sheetfile" "pcb.kicad_sch")
     (property "Sheetname" "")
     (property "ki_description" "Resistor")
@@
     (descr "Resistor SMD 1206 (3216 Metric), square (rectangular) end terminal, IPC_7351 nominal with elongated pad for handsoldering. (Body size source: IPC-SM-782 page 72, https://www.pcb-3d.com/wordpress/wp-content/uploads/ipc-sm-782a_amendment_1_and_2.pdf), generated with kicad-footprint-generator")
     (tags "resistor handsolder")
-    (property "Sheetfile" "qsolder_pcb.kicad_sch")
+    (property "Sheetfile" "pcb.kicad_sch")
     (property "Sheetname" "")
     (property "ki_description" "Resistor")
@@
     (descr "Capacitor SMD 1206 (3216 Metric), square (rectangular) end terminal, IPC_7351 nominal with elongated pad for handsoldering. (Body size source: IPC-SM-782 page 76, https://www.pcb-3d.com/wordpress/wp-content/uploads/ipc-sm-782a_amendment_1_and_2.pdf), generated with kicad-footprint-generator")
     (tags "capacitor handsolder")
-    (property "Sheetfile" "qsolder_pcb.kicad_sch")
+    (property "Sheetfile" "pcb.kicad_sch")
     (property "Sheetname" "")
     (property "ki_description" "Unpolarized capacitor")
@@
     (descr "LQFP, 48 Pin (https://www.analog.com/media/en/technical-documentation/data-sheets/ltc2358-16.pdf), generated with kicad-footprint-generator ipc_gullwing_generator.py")
     (tags "LQFP QFP")
-    (property "Sheetfile" "qsolder_pcb.kicad_sch")
+    (property "Sheetfile" "pcb.kicad_sch")
     (property "Sheetname" "")
     (property "ki_description" "ARM Cortex-M3 MCU, 128KB flash, 20KB RAM, 72MHz, 2-3.6V, 37 GPIO, LQFP-48")
@@
     (descr "Capacitor SMD 1206 (3216 Metric), square (rectangular) end terminal, IPC_7351 nominal with elongated pad for handsoldering. (Body size source: IPC-SM-782 page 76, https://www.pcb-3d.com/wordpress/wp-content/uploads/ipc-sm-782a_amendment_1_and_2.pdf), generated with kicad-footprint-generator")
     (tags "capacitor handsolder")
-    (property "Sheetfile" "qsolder_pcb.kicad_sch")
+    (property "Sheetfile" "pcb.kicad_sch")
     (property "Sheetname" "")
     (property "ki_description" "Unpolarized capacitor")
@@
     (descr "SOIC, 8 Pin (JEDEC MS-012AA, https://www.analog.com/media/en/package-pcb-resources/package/pkg_pdf/soic_narrow-r/r_8.pdf), generated with kicad-footprint-generator ipc_gullwing_generator.py")
     (tags "SOIC SO")
-    (property "Sheetfile" "qsolder_pcb.kicad_sch")
+    (property "Sheetfile" "pcb.kicad_sch")
     (property "Sheetname" "")
     (property "ki_description" "64Kb serial FRAM nonvolatile Memory, SOIC-8")
@@
     (descr "Capacitor SMD 1206 (3216 Metric), square (rectangular) end terminal, IPC_7351 nominal with elongated pad for handsoldering. (Body size source: IPC-SM-782 page 76, https://www.pcb-3d.com/wordpress/wp-content/uploads/ipc-sm-782a_amendment_1_and_2.pdf), generated with kicad-footprint-generator")
     (tags "capacitor handsolder")
-    (property "Sheetfile" "qsolder_pcb.kicad_sch")
+    (property "Sheetfile" "pcb.kicad_sch")
     (property "Sheetname" "")
     (property "ki_description" "Unpolarized capacitor")
@@
     (descr "Capacitor SMD 1206 (3216 Metric), square (rectangular) end terminal, IPC_7351 nominal with elongated pad for handsoldering. (Body size source: IPC-SM-782 page 76, https://www.pcb-3d.com/wordpress/wp-content/uploads/ipc-sm-782a_amendment_1_and_2.pdf), generated with kicad-footprint-generator")
     (tags "capacitor handsolder")
-    (property "Sheetfile" "qsolder_pcb.kicad_sch")
+    (property "Sheetfile" "pcb.kicad_sch")
     (property "Sheetname" "")
     (property "ki_description" "Unpolarized capacitor")
