File: pcb/power.kicad_sch (KiCad schematic)
At the start: 27 parts, among them J18 24v, J20 POWER_BTN, J3 POWER_BTN_MCU, J4 220, J4 220_OUT, Q9 BCX56, U8 MC34063AD, U9 H11AA1

Commit message: Change resistense on R46 to 1k (add raleay on more power)
Parts:
- R46: value 10k -> 1k
Changed lines of the file:
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@@
     (pin "2")
     (instances
-      (project "qsolder_pcb"
+      (project "pcb"
         (path "/484c7117-151d-4c67-9cf5-351046124522/9e093e5e-7e4e-4b34-9a62-04ff3d66b5a3"
           (reference "L2") (unit 1)
@@
     (pin "1")
     (instances
-      (project "qsolder_pcb"
+      (project "pcb"
         (path "/484c7117-151d-4c67-9cf5-351046124522/9e093e5e-7e4e-4b34-9a62-04ff3d66b5a3"
           (reference "#PWR061") (unit 1)
@@
     (pin "2")
     (instances
-      (project "qsolder_pcb"
+      (project "pcb"
         (path "/484c7117-151d-4c67-9cf5-351046124522/9e093e5e-7e4e-4b34-9a62-04ff3d66b5a3"
           (reference "C22") (unit 1)
@@
     (pin "1")
     (instances
-      (project "qsolder_pcb"
+      (project "pcb"
         (path "/484c7117-151d-4c67-9cf5-351046124522/9e093e5e-7e4e-4b34-9a62-04ff3d66b5a3"
           (reference "#PWR058") (unit 1)
@@
     (pin "1")
     (instances
-      (project "qsolder_pcb"
+      (project "pcb"
         (path "/484c7117-151d-4c67-9cf5-351046124522/9e093e5e-7e4e-4b34-9a62-04ff3d66b5a3"
           (reference "#PWR064") (unit 1)
@@
     (pin "1")
     (instances
-      (project "qsolder_pcb"
+      (project "pcb"
         (path "/484c7117-151d-4c67-9cf5-351046124522/9e093e5e-7e4e-4b34-9a62-04ff3d66b5a3"
           (reference "#PWR0109") (unit 1)
@@
     (pin "2")
     (instances
-      (project "qsolder_pcb"
+      (project "pcb"
         (path "/484c7117-151d-4c67-9cf5-351046124522/9e093e5e-7e4e-4b34-9a62-04ff3d66b5a3"
           (reference "D5") (unit 1)
@@
     (pin "5")
     (instances
-      (project "qsolder_pcb"
+      (project "pcb"
         (path "/484c7117-151d-4c67-9cf5-351046124522/9e093e5e-7e4e-4b34-9a62-04ff3d66b5a3"
           (reference "Relay1") (unit 1)
@@
     (pin "2")
     (instances
-      (project "qsolder_pcb"
+      (project "pcb"
         (path "/484c7117-151d-4c67-9cf5-351046124522/9e093e5e-7e4e-4b34-9a62-04ff3d66b5a3"
           (reference "J20") (unit 1)
@@
     (pin "2")
     (instances
-      (project "qsolder_pcb"
+      (project "pcb"
         (path "/484c7117-151d-4c67-9cf5-351046124522/9e093e5e-7e4e-4b34-9a62-04ff3d66b5a3"
           (reference "C26") (unit 1)
@@
     (pin "1")
     (instances
-      (project "qsolder_pcb"
+      (project "pcb"
         (path "/484c7117-151d-4c67-9cf5-351046124522/9e093e5e-7e4e-4b34-9a62-04ff3d66b5a3"
           (reference "#PWR063") (unit 1)
@@
     (pin "1")
     (instances
-      (project "qsolder_pcb"
+      (project "pcb"
         (path "/484c7117-151d-4c67-9cf5-351046124522/9e093e5e-7e4e-4b34-9a62-04ff3d66b5a3"
           (reference "#PWR060") (unit 1)
@@
     (pin "6")
     (instances
-      (project "qsolder_pcb"
+      (project "pcb"
         (path "/484c7117-151d-4c67-9cf5-351046124522/9e093e5e-7e4e-4b34-9a62-04ff3d66b5a3"
           (reference "U9") (unit 1)
@@
     (pin "1")
     (instances
-      (project "qsolder_pcb"
+      (project "pcb"
         (path "/484c7117-151d-4c67-9cf5-351046124522/9e093e5e-7e4e-4b34-9a62-04ff3d66b5a3"
           (reference "#PWR057") (unit 1)
@@
     (pin "1")
     (instances
-      (project "qsolder_pcb"
+      (project "pcb"
         (path "/484c7117-151d-4c67-9cf5-351046124522/9e093e5e-7e4e-4b34-9a62-04ff3d66b5a3"
           (reference "#PWR067") (unit 1)
@@
     (pin "8")
     (instances
-      (project "qsolder_pcb"
+      (project "pcb"
         (path "/484c7117-151d-4c67-9cf5-351046124522/9e093e5e-7e4e-4b34-9a62-04ff3d66b5a3"
           (reference "U8") (unit 1)
@@
     (pin "1")
     (instances
-      (project "qsolder_pcb"
+      (project "pcb"
         (path "/484c7117-151d-4c67-9cf5-351046124522/9e093e5e-7e4e-4b34-9a62-04ff3d66b5a3"
           (reference "#PWR062") (unit 1)
@@
     (pin "2")
     (instances
-      (project "qsolder_pcb"
+      (project "pcb"
         (path "/484c7117-151d-4c67-9cf5-351046124522/9e093e5e-7e4e-4b34-9a62-04ff3d66b5a3"
           (reference "R6") (unit 1)
@@
     (pin "2")
     (instances
-      (project "qsolder_pcb"
+      (project "pcb"
         (path "/484c7117-151d-4c67-9cf5-351046124522/9e093e5e-7e4e-4b34-9a62-04ff3d66b5a3"
           (reference "J3") (unit 1)
@@
     (pin "1")
     (instances
-      (project "qsolder_pcb"
+      (project "pcb"
         (path "/484c7117-151d-4c67-9cf5-351046124522/9e093e5e-7e4e-4b34-9a62-04ff3d66b5a3"
           (reference "#PWR04") (unit 1)
@@
     (pin "2")
     (instances
-      (project "qsolder_pcb"
+      (project "pcb"
         (path "/484c7117-151d-4c67-9cf5-351046124522/9e093e5e-7e4e-4b34-9a62-04ff3d66b5a3"
           (reference "C21") (unit 1)
@@
     (pin "2")
     (instances
-      (project "qsolder_pcb"
+      (project "pcb"
         (path "/484c7117-151d-4c67-9cf5-351046124522/9e093e5e-7e4e-4b34-9a62-04ff3d66b5a3"
           (reference "R53") (unit 1)
@@
     (pin "2")
     (instances
-      (project "qsolder_pcb"
+      (project "pcb"
         (path "/484c7117-151d-4c67-9cf5-351046124522/9e093e5e-7e4e-4b34-9a62-04ff3d66b5a3"
           (reference "R54") (unit 1)
@@
     (pin "2")
     (instances
-      (project "qsolder_pcb"
+      (project "pcb"
         (path "/484c7117-151d-4c67-9cf5-351046124522/9e093e5e-7e4e-4b34-9a62-04ff3d66b5a3"
           (reference "R52") (unit 1)
@@
     (pin "1")
     (instances
-      (project "qsolder_pcb"
+      (project "pcb"
         (path "/484c7117-151d-4c67-9cf5-351046124522/9e093e5e-7e4e-4b34-9a62-04ff3d66b5a3"
           (reference "#PWR05") (unit 1)
@@
     (pin "2")
     (instances
-      (project "qsolder_pcb"
+      (project "pcb"
         (path "/484c7117-151d-4c67-9cf5-351046124522/9e093e5e-7e4e-4b34-9a62-04ff3d66b5a3"
           (reference "J18") (unit 1)
@@
     (pin "2")
     (instances
-      (project "qsolder_pcb"
+      (project "pcb"
         (path "/484c7117-151d-4c67-9cf5-351046124522/9e093e5e-7e4e-4b34-9a62-04ff3d66b5a3"
           (reference "R44") (unit 1)
@@
       (effects (font (size 1.27 1.27)))
     )
-    (property "Value" "10k" (at 188.595 45.085 90)
+    (property "Value" "1k" (at 188.595 45.085 90)
       (effects (font (size 1.27 1.27)))
     )
@@
     (pin "2")
     (instances
-      (project "qsolder_pcb"
+      (project "pcb"
         (path "/484c7117-151d-4c67-9cf5-351046124522/9e093e5e-7e4e-4b34-9a62-04ff3d66b5a3"
           (reference "R46") (unit 1)
@@
     (pin "2")
     (instances
-      (project "qsolder_pcb"
+      (project "pcb"
         (path "/484c7117-151d-4c67-9cf5-351046124522/9e093e5e-7e4e-4b34-9a62-04ff3d66b5a3"
           (reference "C27") (unit 1)
@@
     (pin "2")
     (instances
-      (project "qsolder_pcb"
+      (project "pcb"
         (path "/484c7117-151d-4c67-9cf5-351046124522/9e093e5e-7e4e-4b34-9a62-04ff3d66b5a3"
           (reference "L1") (unit 1)
@@
     (pin "3")
     (instances
-      (project "qsolder_pcb"
+      (project "pcb"
         (path "/484c7117-151d-4c67-9cf5-351046124522/9e093e5e-7e4e-4b34-9a62-04ff3d66b5a3"
           (reference "Q9") (unit 1)
@@
     (pin "2")
     (instances
-      (project "qsolder_pcb"
+      (project "pcb"
         (path "/484c7117-151d-4c67-9cf5-351046124522/9e093e5e-7e4e-4b34-9a62-04ff3d66b5a3"
           (reference "R43") (unit 1)
@@
     (pin "1")
     (instances
-      (project "qsolder_pcb"
+      (project "pcb"
         (path "/484c7117-151d-4c67-9cf5-351046124522/9e093e5e-7e4e-4b34-9a62-04ff3d66b5a3"
           (reference "#PWR066") (unit 1)
@@
     (pin "1")
     (instances
-      (project "qsolder_pcb"
+      (project "pcb"
         (path "/484c7117-151d-4c67-9cf5-351046124522/9e093e5e-7e4e-4b34-9a62-04ff3d66b5a3"
           (reference "#FLG02") (unit 1)
@@
     (pin "2")
     (instances
-      (project "qsolder_pcb"
+      (project "pcb"
         (path "/484c7117-151d-4c67-9cf5-351046124522/9e093e5e-7e4e-4b34-9a62-04ff3d66b5a3"
           (reference "C25") (unit 1)
@@
     (pin "1")
     (instances
-      (project "qsolder_pcb"
+      (project "pcb"
         (path "/484c7117-151d-4c67-9cf5-351046124522/9e093e5e-7e4e-4b34-9a62-04ff3d66b5a3"
           (reference "#PWR059") (unit 1)
@@
     (pin "1")
     (instances
-      (project "qsolder_pcb"
+      (project "pcb"
         (path "/484c7117-151d-4c67-9cf5-351046124522/9e093e5e-7e4e-4b34-9a62-04ff3d66b5a3"
           (reference "#PWR0107") (unit 1)
@@
     (pin "2")
     (instances
-      (project "qsolder_pcb"
+      (project "pcb"
         (path "/484c7117-151d-4c67-9cf5-351046124522/9e093e5e-7e4e-4b34-9a62-04ff3d66b5a3"
           (reference "R45") (unit 1)
@@
     (pin "2")
     (instances
-      (project "qsolder_pcb"
+      (project "pcb"
         (path "/484c7117-151d-4c67-9cf5-351046124522"
           (reference "J4") (unit 1)
@@
     (pin "1")
     (instances
-      (project "qsolder_pcb"
+      (project "pcb"
         (path "/484c7117-151d-4c67-9cf5-351046124522/9e093e5e-7e4e-4b34-9a62-04ff3d66b5a3"
           (reference "#PWR065") (unit 1)
@@
     (pin "2")
     (instances
-      (project "qsolder_pcb"
+      (project "pcb"
         (path "/484c7117-151d-4c67-9cf5-351046124522"
           (reference "J4") (unit 1)
@@
     (pin "2")
     (instances
-      (project "qsolder_pcb"
+      (project "pcb"
         (path "/484c7117-151d-4c67-9cf5-351046124522/9e093e5e-7e4e-4b34-9a62-04ff3d66b5a3"
           (reference "C24") (unit 1)
@@
     (pin "2")
     (instances
-      (project "qsolder_pcb"
+      (project "pcb"
         (path "/484c7117-151d-4c67-9cf5-351046124522/9e093e5e-7e4e-4b34-9a62-04ff3d66b5a3"
           (reference "D4") (unit 1)
@@
     (pin "1")
     (instances
-      (project "qsolder_pcb"
+      (project "pcb"
         (path "/484c7117-151d-4c67-9cf5-351046124522/9e093e5e-7e4e-4b34-9a62-04ff3d66b5a3"
           (reference "#FLG01") (unit 1)
